File: hw/sch_pcb/USTSIPIN03.kicad_pcb (KiCad board)
At the start: 2 copper layers, 70.6 x 50.3 mm, 107 parts, among them J1 HEADER_2x15, M1 HOLE, M2 HOLE, M3 HOLE, M4 HOLE, M5 RFShield_TwoPieces, Q1 2SK2394-6, U1 ISL21080CIH341Z-TK, U10 ISL21080DIH309, U11 AT24CS64-SSHM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

Commit message: Update Kicad project version.
Parts:
- C15: value 2n2 -> 3n3
Changed lines of the file:
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@@
     (property "Sheetfile" "analogue_backend.kicad_sch")
     (property "Sheetname" "analogue_backend")
-    (property "UST_ID" "5c70984712875079b91f8b46")
+    (property "UST_ID" "651abc26462c6d9e720551fa")
     (property "ki_description" "Unpolarized capacitor")
     (property "ki_keywords" "cap capacitor")
@@
         (effects (font (size 1 1) (thickness 0.15)) (justify mirror))
     )
-    (fp_text value "2n2" (at 0 -1.68 90) (layer "B.Fab") hide
+    (fp_text value "3n3" (at 0 -1.68 90) (layer "B.Fab") hide
         (effects (font (size 1 1) (thickness 0.15)) (justify mirror))
     )
@@
     (property "Sheetfile" "interface.kicad_sch")
     (property "Sheetname" "interface")
-    (property "UST_ID" "5c70984812875079b91f8bbe")
+    (property "UST_ID" "5c70984712875079b91f8b53")
     (property "ki_description" "Unpolarized capacitor")
     (property "ki_keywords" "cap capacitor")
@@
     (property "Sheetfile" "interface.kicad_sch")
     (property "Sheetname" "interface")
-    (property "UST_ID" "5c70984812875079b91f8bbe")
-    (property "UST_id" "")
+    (property "UST_ID" "5c70984712875079b91f8b53")
     (property "ki_description" "Unpolarized capacitor, small symbol")
     (property "ki_keywords" "capacitor cap")
