File: hw/sch_pcb/USTSIPIN03.kicad_sch (KiCad schematic)
At the start: 8 parts, among them M1 HOLE, M2 HOLE, M3 HOLE, M4 HOLE

Commit message: Update silkscreen and title blocks.
Other:
- title: AIRDOS04A base board -> USTSIPIN03A
Changed lines of the file:
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@@
   (paper "A4")
   (title_block
-    (title "AIRDOS04A base board")
-    (date "2023-10-23")
+    (title "USTSIPIN03A")
+    (date "2023-11-13")
     (company "Jakub Kákona <info@ust.cz>")
-    (comment 2 "Airborne semiconductor\\nionizing radiation detector")
+    (comment 2 "Semiconductor\\nionizing radiation detector")
     (comment 4 "GPL 3")
   )
@@
     (pin "1")
     (instances
-      (project "AIRDOS04_sensor"
+      (project "USTSIPIN03"
         (path "/e63e39d7-6ac0-4ffd-8aa3-1841a4541b55"
           (reference "M1") (unit 1)
@@
         )
       )
-      (project "AIRDOS04_sensor"
+      (project "USTSIPIN03"
         (path "/e63e39d7-6ac0-4ffd-8aa3-1841a4541b55/e191f86f-5b54-4b8b-aca6-37b81226f3b6"
           (reference "FID4") (unit 1)
@@
         )
       )
-      (project "AIRDOS04_sensor"
+      (project "USTSIPIN03"
         (path "/e63e39d7-6ac0-4ffd-8aa3-1841a4541b55/e191f86f-5b54-4b8b-aca6-37b81226f3b6"
           (reference "FID3") (unit 1)
@@
     (pin "1")
     (instances
-      (project "AIRDOS04_sensor"
+      (project "USTSIPIN03"
         (path "/e63e39d7-6ac0-4ffd-8aa3-1841a4541b55"
           (reference "#PWR01") (unit 1)
@@
     (pin "1")
     (instances
-      (project "AIRDOS04_sensor"
+      (project "USTSIPIN03"
         (path "/e63e39d7-6ac0-4ffd-8aa3-1841a4541b55"
           (reference "M2") (unit 1)
@@
     (pin "1")
     (instances
-      (project "AIRDOS04_sensor"
+      (project "USTSIPIN03"
         (path "/e63e39d7-6ac0-4ffd-8aa3-1841a4541b55"
           (reference "M3") (unit 1)
@@
     )
     (instances
-      (project "AIRDOS04_sensor"
+      (project "USTSIPIN03"
         (path "/e63e39d7-6ac0-4ffd-8aa3-1841a4541b55"
           (reference "FID1") (unit 1)
@@
     )
     (instances
-      (project "AIRDOS04_sensor"
+      (project "USTSIPIN03"
         (path "/e63e39d7-6ac0-4ffd-8aa3-1841a4541b55"
           (reference "FID2") (unit 1)
@@
     (pin "1")
     (instances
-      (project "AIRDOS04_sensor"
+      (project "USTSIPIN03"
         (path "/e63e39d7-6ac0-4ffd-8aa3-1841a4541b55"
           (reference "M4") (unit 1)
@@
     )
     (instances
-      (project "AIRDOS04_sensor"
+      (project "USTSIPIN03"
         (path "/e63e39d7-6ac0-4ffd-8aa3-1841a4541b55" (page "4"))
       )
@@
     )
     (instances
-      (project "AIRDOS04_sensor"
+      (project "USTSIPIN03"
         (path "/e63e39d7-6ac0-4ffd-8aa3-1841a4541b55" (page "2"))
       )
@@
     )
     (instances
-      (project "AIRDOS04_sensor"
+      (project "USTSIPIN03"
         (path "/e63e39d7-6ac0-4ffd-8aa3-1841a4541b55" (page "3"))
       )

Commit message: Fix USTID
Parts:
- FID1, FID2: now left out of the parts list
Changed lines of the file:
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@@
   )
   (symbol (lib_id "Mechanical:Fiducial") (at 264.16 43.18 0) (unit 1)
-    (in_bom yes) (on_board yes) (dnp no) (fields_autoplaced)
+    (in_bom no) (on_board yes) (dnp no) (fields_autoplaced)
     (property "Reference" "FID2" (at 266.319 41.9679 0)
       (effects (font (size 1.27 1.27)) (justify left))
@@
     )
     (property "Datasheet" "~" (at 264.16 43.18 0)
+      (effects (font (size 1.27 1.27)) hide)
+    )
+    (property "UST_ID" "" (at 264.16 43.18 0)
       (effects (font (size 1.27 1.27)) hide)
     )
@@
   )
   (symbol (lib_id "Mechanical:Fiducial") (at 251.46 43.18 0) (unit 1)
-    (in_bom yes) (on_board yes) (dnp no) (fields_autoplaced)
+    (in_bom no) (on_board yes) (dnp no) (fields_autoplaced)
     (property "Reference" "FID1" (at 253.619 41.9679 0)
       (effects (font (size 1.27 1.27)) (justify left))
@@
     )
     (property "Datasheet" "~" (at 251.46 43.18 0)
+      (effects (font (size 1.27 1.27)) hide)
+    )
+    (property "UST_ID" "" (at 251.46 43.18 0)
       (effects (font (size 1.27 1.27)) hide)
     )
@@
   )
   (symbol (lib_id "Mechanical:Fiducial") (at 251.46 36.83 0) (unit 1)
-    (in_bom yes) (on_board yes) (dnp no) (fields_autoplaced)
+    (in_bom no) (on_board yes) (dnp no) (fields_autoplaced)
     (property "Reference" "FID1" (at 253.619 35.6179 0)
       (effects (font (size 1.27 1.27)) (justify left))
@@
     )
     (property "Datasheet" "~" (at 251.46 36.83 0)
+      (effects (font (size 1.27 1.27)) hide)
+    )
+    (property "UST_ID" "" (at 251.46 36.83 0)
       (effects (font (size 1.27 1.27)) hide)
     )
@@
   )
   (symbol (lib_id "Mechanical:Fiducial") (at 264.16 36.83 0) (unit 1)
-    (in_bom yes) (on_board yes) (dnp no) (fields_autoplaced)
+    (in_bom no) (on_board yes) (dnp no) (fields_autoplaced)
     (property "Reference" "FID2" (at 266.319 35.6179 0)
       (effects (font (size 1.27 1.27)) (justify left))
@@
       (effects (font (size 1.27 1.27)) hide)
     )
+    (property "UST_ID" "" (at 264.16 36.83 0)
+      (effects (font (size 1.27 1.27)) hide)
+    )

Commit message: Update Kicad project version.
Other:
- company: Jakub Kákona <info@ust.cz> -> kaklik <info@ust.cz>
- title: USTSIPIN03A -> USTSIPIN03B
Changed lines of the file:
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@@
   (paper "A4")
   (title_block
-    (title "USTSIPIN03A")
-    (date "2023-11-13")
-    (company "Jakub Kákona <info@ust.cz>")
+    (title "USTSIPIN03B")
+    (date "2024-05-30")
+    (company "kaklik <info@ust.cz>")
     (comment 2 "Semiconductor\\nionizing radiation detector")
     (comment 4 "GPL 3")
@@
         (path "/e63e39d7-6ac0-4ffd-8aa3-1841a4541b55"
           (reference "M1") (unit 1)
-        )
-        (path "/e63e39d7-6ac0-4ffd-8aa3-1841a4541b55/5c006114-f78d-4936-a365-c4e7307459e1"
-          (reference "M2") (unit 1)
         )
       )
@@
       )
       (project "USTSIPIN03"
-        (path "/e63e39d7-6ac0-4ffd-8aa3-1841a4541b55/e191f86f-5b54-4b8b-aca6-37b81226f3b6"
-          (reference "FID4") (unit 1)
-        )
         (path "/e63e39d7-6ac0-4ffd-8aa3-1841a4541b55"
           (reference "FID4") (unit 1)
@@
       )
       (project "USTSIPIN03"
-        (path "/e63e39d7-6ac0-4ffd-8aa3-1841a4541b55/e191f86f-5b54-4b8b-aca6-37b81226f3b6"
+        (path "/e63e39d7-6ac0-4ffd-8aa3-1841a4541b55"
           (reference "FID3") (unit 1)
         )
-        (path "/e63e39d7-6ac0-4ffd-8aa3-1841a4541b55"
-          (reference "FID3") (unit 1)
-        )
       )
     )
@@
           (reference "#PWR01") (unit 1)
         )
-        (path "/e63e39d7-6ac0-4ffd-8aa3-1841a4541b55/5c006114-f78d-4936-a365-c4e7307459e1"
-          (reference "#PWR016") (unit 1)
-        )
       )
     )
@@
           (reference "M2") (unit 1)
         )
-        (path "/e63e39d7-6ac0-4ffd-8aa3-1841a4541b55/5c006114-f78d-4936-a365-c4e7307459e1"
+      )
+    )
+  )
+  (symbol (lib_id "MLAB_MECHANICAL:HOLE") (at 265.43 24.13 90) (unit 1)
+    (in_bom yes) (on_board yes) (dnp no)
+    (property "Reference" "M3" (at 265.43 26.67 90)
+      (effects (font (size 1.524 1.524)))
+    )
+    (property "Value" "HOLE" (at 267.97 24.13 0)
+      (effects (font (size 1.524 1.524)) hide)
+    )
+    (property "Footprint" "Mlab_Mechanical:MountingHole_3mm" (at 265.43 24.13 0)
+      (effects (font (size 1.524 1.524)) hide)
+    )
+    (property "Datasheet" "" (at 265.43 24.13 0)
+      (effects (font (size 1.524 1.524)))
+    )
+    (pin "1")
+    (instances
+      (project "USTSIPIN03"
+        (path "/e63e39d7-6ac0-4ffd-8aa3-1841a4541b55"
           (reference "M3") (unit 1)
-        )
-      )
-    )
-  )
-  (symbol (lib_id "MLAB_MECHANICAL:HOLE") (at 265.43 24.13 90) (unit 1)
-    (in_bom yes) (on_board yes) (dnp no)
-    (property "Reference" "M3" (at 265.43 26.67 90)
-      (effects (font (size 1.524 1.524)))
-    )
-    (property "Value" "HOLE" (at 267.97 24.13 0)
-      (effects (font (size 1.524 1.524)) hide)
-    )
-    (property "Footprint" "Mlab_Mechanical:MountingHole_3mm" (at 265.43 24.13 0)
-      (effects (font (size 1.524 1.524)) hide)
-    )
-    (property "Datasheet" "" (at 265.43 24.13 0)
-      (effects (font (size 1.524 1.524)))
-    )
-    (pin "1")
-    (instances
-      (project "USTSIPIN03"
-        (path "/e63e39d7-6ac0-4ffd-8aa3-1841a4541b55"
-          (reference "M3") (unit 1)
-        )
-        (path "/e63e39d7-6ac0-4ffd-8aa3-1841a4541b55/5c006114-f78d-4936-a365-c4e7307459e1"
-          (reference "M4") (unit 1)
         )
       )
@@
           (reference "FID1") (unit 1)
         )
-        (path "/e63e39d7-6ac0-4ffd-8aa3-1841a4541b55/5c006114-f78d-4936-a365-c4e7307459e1"
-          (reference "FID1") (unit 1)
-        )
       )
     )
@@
           (reference "FID2") (unit 1)
         )
-        (path "/e63e39d7-6ac0-4ffd-8aa3-1841a4541b55/5c006114-f78d-4936-a365-c4e7307459e1"
-          (reference "FID2") (unit 1)
-        )
       )
     )
@@
           (reference "M4") (unit 1)
         )
-        (path "/e63e39d7-6ac0-4ffd-8aa3-1841a4541b55/5c006114-f78d-4936-a365-c4e7307459e1"
-          (reference "M5") (unit 1)
-        )
-      )
+      )
