File: hw/sch_pcb/analogue_backend.kicad_sch (KiCad schematic)
At the start: 37 parts, among them M5 RFShield_TwoPieces, U1 TS3021ILT, U2 AD8691, U3 ISL21080CIH341Z-TK, U3 LTC1865-MS, U5 SN74LVC2G74, U6 AD8691

Commit message: Update silkscreen and title blocks.
Other:
- title: AIRDOS04A base board -> USTSIPIN03A

Commit message: Fix USTID
Parts:
- C13: UST_ID 6508260b462c6d9e720541f1 -> 5c70984712875079b91f8b4c
- C59: UST_ID 5c70984812875079b91f8bf2 -> 5c70984712875079b91f8b4c
Changed lines of the file:
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@@
       (effects (font (size 1.27 1.27)) hide)
     )
-    (property "UST_ID" "6508260b462c6d9e720541f1" (at 199.39 124.46 0)
+    (property "UST_ID" "5c70984712875079b91f8b4c" (at 199.39 124.46 0)
       (effects (font (size 1.27 1.27)) hide)
     )
@@
       (effects (font (size 1.27 1.27)) hide)
     )
-    (property "UST_ID" "5c70984812875079b91f8bf2" (at 257.81 76.2 0)
+    (property "UST_ID" "5c70984712875079b91f8b4c" (at 257.81 76.2 0)
       (effects (font (size 1.27 1.27)) hide)
     )
@@
       (effects (font (size 1.27 1.27)) hide)
     )
-    (property "UST_ID" "5c70984812875079b91f8bf2" (at 191.77 67.31 0)
-      (effects (font (size 1.27 1.27)) hide)
-    )
+    (property "UST_ID" "5c70984712875079b91f8b4c" (at 191.77 67.31 0)
+      (effects (font (size 1.27 1.27)) hide)
+    )

Commit message: FIX USTIDs.
Parts:
- C19: UST_ID 5d47bf10128750448e6b4652 -> 5c70984812875079b91f8ba6
- C19: value 1nF NP0 -> 1nF; UST_ID 5d47bf10128750448e6b4652 -> 5c70984812875079b91f8ba6
- R11: UST_ID (none) -> 5c70984612875079b91f899f
- U3: UST_ID (none) -> 651eaece462c6d9e72055763
- U3: UST_ID (none) -> 6555591d0c8d609e3e79abc1
- U5: UST_ID (none) -> 65555d4795a79cc5ac409b41
Changed lines of the file:
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@@
       (effects (font (size 1.27 1.27)) hide)
     )
-    (property "UST_ID" "" (at 93.98 99.06 0)
+    (property "UST_ID" "5c70984612875079b91f899f" (at 93.98 99.06 0)
       (effects (font (size 1.27 1.27)) hide)
     )
@@
       (effects (font (size 1.27 1.27)) hide)
     )
-    (property "UST_ID" "" (at 189.23 142.24 0)
+    (property "UST_ID" "65555d4795a79cc5ac409b41" (at 189.23 142.24 0)
       (effects (font (size 1.27 1.27)) hide)
     )
@@
     )
     (property "Datasheet" "https://www.analog.com/media/en/technical-documentation/data-sheets/18645fb.pdf" (at 242.57 104.14 0)
+      (effects (font (size 1.27 1.27)) hide)
+    )
+    (property "UST_ID" "651eaece462c6d9e72055763" (at 242.57 104.14 0)
       (effects (font (size 1.27 1.27)) hide)
     )
@@
       (effects (font (size 1.27 1.27)) hide)
     )
-    (property "UST_ID" "" (at 133.35 99.06 0)
+    (property "UST_ID" "5c70984612875079b91f899f" (at 133.35 99.06 0)
       (effects (font (size 1.27 1.27)) hide)
     )
@@
       (effects (font (size 1.27 1.27) italic) hide)
     )
-    (property "UST_ID" "" (at 203.2 69.85 0)
+    (property "UST_ID" "6555591d0c8d609e3e79abc1" (at 203.2 69.85 0)
       (effects (font (size 1.27 1.27)) hide)
     )
@@
       (effects (font (size 1.27 1.27)) hide)
     )
-    (property "UST_ID" "5d47bf10128750448e6b4652" (at 218.44 111.76 0)
+    (property "UST_ID" "5c70984812875079b91f8ba6" (at 218.44 111.76 0)
       (effects (font (size 1.27 1.27)) hide)
     )
@@
       (effects (font (size 1.27 1.27)) (justify left))
     )
-    (property "Value" "1nF NP0" (at 138.43 96.52 0)
+    (property "Value" "1nF" (at 137.16 101.6 0)
       (effects (font (size 1.27 1.27)) (justify left))
     )
@@
       (effects (font (size 1.27 1.27)) hide)
     )
-    (property "UST_ID" "5d47bf10128750448e6b4652" (at 142.24 104.14 0)
-      (effects (font (size 1.27 1.27)) hide)
-    )
+    (property "UST_ID" "5c70984812875079b91f8ba6" (at 142.24 104.14 0)
+      (effects (font (size 1.27 1.27)) hide)
+    )

Commit message: Add notes to power consumption.
Other:
- note added: "+1.2 mA"
- note added: "+1.3 mA max"
- note added: "10 μA"
- note added: "73 μA"
Changed lines of the file:
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@@
     (stroke (width 0) (type solid))
+  )
+  (text "+1.3 mA max" (at 242.57 68.58 0)
+    (effects (font (size 1.524 1.524)) (justify left bottom))
+  )
+  (text "+1.2 mA" (at 81.28 74.93 0)
+    (effects (font (size 1.524 1.524)) (justify left bottom))
+  )
+  (text "73 μA" (at 82.55 48.26 0)
+    (effects (font (size 1.524 1.524)) (justify left bottom))
+  )
+  (text "+1.2 mA" (at 83.82 21.59 0)
+    (effects (font (size 1.524 1.524)) (justify left bottom))
+  )
+  (text "10 μA" (at 190.5 118.11 0)
+    (effects (font (size 1.524 1.524)) (justify left bottom))
   )
   (label "VCC3" (at 83.82 52.07 0) (fields_autoplaced)

Commit message: Removed hand-soldering footprints for OpAmps. Rosolve #1
Parts:
- U1: footprint Package_TO_SOT_SMD:SOT-23-5_HandSoldering -> Package_TO_SOT_SMD:SOT-23-5
- U2, U6: footprint Package_TO_SOT_SMD:TSOT-23-5_HandSoldering -> Package_TO_SOT_SMD:TSOT-23-5
Changed lines of the file:
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@@
       (effects (font (size 1.27 1.27)) (justify left))
     )
-    (property "Footprint" "Package_TO_SOT_SMD:SOT-23-5_HandSoldering" (at 149.86 144.78 0)
+    (property "Footprint" "Package_TO_SOT_SMD:SOT-23-5" (at 149.86 144.78 0)
       (effects (font (size 1.27 1.27)) hide)
     )
@@
       (effects (font (size 1.27 1.27)) (justify left))
     )
-    (property "Footprint" "Package_TO_SOT_SMD:TSOT-23-5_HandSoldering" (at 95.25 114.3 0)
+    (property "Footprint" "Package_TO_SOT_SMD:TSOT-23-5" (at 95.25 114.3 0)
       (effects (font (size 1.27 1.27)) hide)
     )
@@
       (effects (font (size 1.27 1.27)) (justify left))
     )
-    (property "Footprint" "Package_TO_SOT_SMD:TSOT-23-5_HandSoldering" (at 168.91 101.6 0)
-      (effects (font (size 1.27 1.27)) hide)
-    )
+    (property "Footprint" "Package_TO_SOT_SMD:TSOT-23-5" (at 168.91 101.6 0)
+      (effects (font (size 1.27 1.27)) hide)
+    )

Commit message: Uniform capacitor types.
Parts:
- C18: value 2n2 -> 3n3; UST_ID 5c70984712875079b91f8b46 -> 651abc26462c6d9e720551fa
Changed lines of the file:
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@@
       (effects (font (size 1.27 1.27)))
     )
-    (property "Value" "2n2" (at 93.98 87.3506 90)
+    (property "Value" "3n3" (at 93.98 87.3506 90)
       (effects (font (size 1.27 1.27)))
     )
@@
       (effects (font (size 1.27 1.27)) hide)
     )
-    (property "UST_ID" "5c70984712875079b91f8b46" (at 93.98 91.44 0)
+    (property "UST_ID" "651abc26462c6d9e720551fa" (at 93.98 91.44 0)
       (effects (font (size 1.27 1.27)) hide)
     )

Commit message: Update Kicad project version.
Parts:
- renumbered C20 to C10, C3 to C11, C11 to C13, C15 to C14, C19 to C16, C13 to C18, C7 to C3, C12 to C4, C19 to C48, C13 to C7, C3 to C9, R3 to R1, R4 to R2, R9 to R3, R1 to R6, U6 to U4, U1 to U6
Other:
- company: Jakub Kákona <info@ust.cz> -> kaklik <info@ust.cz>
- title: USTSIPIN03A -> USTSIPIN03B
